File: Steckkarte/Steckkarte/Steckkarte.brd (EAGLE design)
At the start: 63 x 92.5 mm, 96 parts, among them IC1 OPA2333D, IC2 TLP2768A_TP,E, U1 STM32L412CBT6, U2 LP5907QMFX-3.3Q1, U3 REF5030AIDR, U4 RFM-0505S, U5 Value, U6 TLV4110IDGNR, U7 W25Q64JVSSIQ, U8 ACSL-6400-00TE, U9 OPA333AIDBVR

Commit message: update layout
Parts:
- moved R16 1.41 mm to (40.2, 11.5)
Connections:
- net MOSI_EXT: no longer R16.1
- net SS_EXT: now also R16.1

Commit message: Fixed some stuff
Parts:
- removed H2: TESTPOINT_TPS-SMD-10SN, 52101-101-REV-A:TESTPOINT_SMD-10SN
- removed R12: 22, rcl:R0603
- added C26: (no value), rcl:C0603K
- added C27, C28, C29, C30: 100n, rcl:C0603K
- R11: value 22 -> 1k
- moved JP2 28.7 mm to (47.7, 48.7), turned to 180 degrees
- moved R17 20.6 mm to (37.0, 30.1)
- moved R11 18.4 mm to (31.0, 45.5), turned to 180 degrees
- moved R21 14.8 mm to (34.3, 8.03), turned to 270 degrees
- moved C16 14.5 mm to (53.8, 44.0)
- moved U7 14.5 mm to (55.0, 38.7), turned to 270 degrees
- moved MISO1 12.3 mm to (35.4, 29.4)
- moved R15 6.53 mm to (46.5, 33.0)
- moved MOSI2 6.36 mm to (47.3, 41.2)
- moved R10 4.49 mm to (46.5, 37.0), turned to 180 degrees
- moved R16 4.02 mm to (38.0, 8.17), turned to 90 degrees
- moved NSS2 3.54 mm to (44.3, 33.0)
- moved MISO2 3.35 mm to (44.1, 39.0)
- moved GND_EXT 3.16 mm to (54.0, 5.00)
- moved R13 3.05 mm to (46.5, 35.0)
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Connections:
- removed net HOLD: H2.TP, R12.1, U1.30
- removed net N$10: R12.2, U7.7
- removed net N$20: IC2.1, R17.1
- removed net N$5: R11.1, U7.3
- removed net WP: R11.2, U1.32
- new net 3.3V_EXT: JP1.15, JP1.16, R16.2, U8.1, U8.3, U8.5, U8.7
- new net 5V_EXT: C17.1, C6.1, IC2.6, JP1.1, JP1.2, JP1.3, JP1.4, U4.1
- new net N$9: R21.1, U8.8
- net +3V3: now also C24.2, IC2.1, R11.2, U1.24, U7.3, U7.7; no longer C24.1, R17.2, U1.23
- net +5V: no longer C17.1, C6.1, IC2.6, JP1.1, JP1.2, JP1.3, JP1.4, R16.2, R21.5, R21.6, R21.7, R21.8, U4.1
- net GND5: now also C24.1, C26.2, C27.2, C28.1, C29.2, C30.1, U1.23, U1.44; no longer C24.2, U1.24
- net MOSI_EXT: now also R21.7; no longer U8.6
- net N$13: now also C30.2
- net N$14: now also C29.1
- net N$15: now also C28.2
- net N$16: now also U8.6; no longer U8.3
- net N$17: now also U8.4; no longer U8.5
- net N$18: now also U8.2; no longer U8.7
- net N$19: now also C26.1, IC2.3, R17.1; no longer R21.1, U8.1
- net RST: now also R11.1
- net SCLK_EXT: now also R21.6; no longer U8.4
- net SF_EXT: now also R21.5; no longer U8.2
- net SPI1_MISO: now also R17.2; no longer IC2.3
- net SPI2_MISO: now also C27.1
- net SS_EXT: now also R21.8; no longer U8.8
Routing:
- net GND5: track 492.6 -> 266.5 mm, vias 123 -> 142
- net +5V: track 304.8 -> 202.6 mm, vias 8 -> 6
- net 5V_EXT: track 0.00 -> 79.2 mm, vias 0 -> 2
- net SWDIO: track 54.4 -> 12.6 mm
- net 3.3V_EXT: track 0.00 -> 41.5 mm, vias 0 -> 1
- net SWCLK: track 37.2 -> 11.3 mm
- net N$10: track 25.6 -> 0.00 mm
- net N$15: track 47.1 -> 23.7 mm
- net N$13: track 31.2 -> 8.35 mm
- net RST: track 49.4 -> 27.9 mm, vias 0 -> 1
- net GND: track 33.2 -> 53.1 mm
- net SPI1_MISO: track 24.2 -> 5.72 mm
- net HOLD: track 13.6 -> 0.00 mm
- net +3V3: track 226.3 -> 213.7 mm, vias 13 -> 10
- net MOSI_EXT: track 14.8 -> 4.71 mm
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- removed copper zone on layer 1, net +5V
Other:
- board text added: "3,3V"
- board text added: "CLK"
- board text added: "DIO"
- board text added: "Gnd"
- board text added: "Nrst"
- board text added: "and partly Johannes Wittmann"
- board text added: "blame Timo Erdmannsdörfer"
