File: Steckkarte/Steckkarte/Steckkarte.sch (EAGLE design)
At the start: 96 parts, among them IC1 OPA2333D, IC2 TLP2768A_TP,E, U1 STM32L412CBT6, U2 LP5907QMFX-3.3Q1, U3 REF5030AIDR, U4 RFM-0505S, U5 Value, U6 TLV4110IDGNR, U7 W25Q64JVSSIQ, U8 ACSL-6400-00TE, U9 OPA333AIDBVR

Commit message: update layout
Connections:
- net MOSI_EXT: no longer R16.1
- net SS_EXT: now also R16.1
Changed lines of the file:
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@@
 <segment>
 <pinref part="U8" gate="A" pin="CATHODE3"/>
-<wire x1="-83.82" y1="-193.04" x2="-99.06" y2="-193.04" width="0.1524" layer="91"/>
+<wire x1="-83.82" y1="-193.04" x2="-96.52" y2="-193.04" width="0.1524" layer="91"/>
 <label x="-93.98" y="-193.04" size="1.778" layer="95"/>
-<pinref part="R16" gate="G$1" pin="1"/>
 </segment>
 </net>
@@
 <segment>
 <pinref part="U8" gate="A" pin="CATHODE4"/>
-<wire x1="-83.82" y1="-195.58" x2="-93.98" y2="-195.58" width="0.1524" layer="91"/>
+<wire x1="-83.82" y1="-195.58" x2="-99.06" y2="-195.58" width="0.1524" layer="91"/>
 <label x="-93.98" y="-195.58" size="1.778" layer="95"/>
+<pinref part="R16" gate="G$1" pin="1"/>
+<wire x1="-99.06" y1="-195.58" x2="-99.06" y2="-193.04" width="0.1524" layer="91"/>
 </segment>
 <segment>

Commit message: Fixed some stuff
Parts:
- removed H2: TESTPOINT_TPS-SMD-10SN, 52101-101-REV-A:TESTPOINT_TPS-SMD-10SN
- removed R12: 22, rcl:R-EU_R0603
- added C26: (no value), rcl:C-EUC0603K
- added C27, C28, C29, C30: 100n, rcl:C-EUC0603K
- R11: value 22 -> 1k
Connections:
- removed net HOLD: H2.TP, R12.1, U1.PA9
- removed net N$10: R12.2, U7./HOLD_OR_/RESET(IO3)
- removed net N$20: IC2.ANODE, R17.1
- removed net N$5: R11.1, U7./WP(IO2)
- removed net WP: R11.2, U1.PA11
- new net 3.3V_EXT: JP1.15, JP1.16, R16.2, U8.ANODE1, U8.ANODE2, U8.ANODE3, U8.ANODE4
- new net 5V_EXT: C17.1, C6.1, IC2.VCC, JP1.1, JP1.2, JP1.3, JP1.4, U4.-VIN
- new net N$9: R21.1, U8.CATHODE4
- net +3V3: now also C24.2, IC2.ANODE, R11.2, U1.VDD_2, U7./HOLD_OR_/RESET(IO3), U7./WP(IO2); no longer C24.1, R17.2, U1.VSS_2
- net +5V: no longer C17.1, C6.1, IC2.VCC, JP1.1, JP1.2, JP1.3, JP1.4, R16.2, R21.5, R21.6, R21.7, R21.8, U4.-VIN
- net GND5: now also C24.1, C26.2, C27.2, C28.1, C29.2, C30.1, U1.PH3/BOOT0, U1.VSS_2; no longer C24.2, U1.VDD_2
- net MOSI_EXT: now also R21.7; no longer U8.CATHODE3
- net N$13: now also C30.2
- net N$14: now also C29.1
- net N$15: now also C28.2
- net N$16: now also U8.CATHODE3; no longer U8.ANODE2
- net N$17: now also U8.CATHODE2; no longer U8.ANODE3
- net N$18: now also U8.CATHODE1; no longer U8.ANODE4
- net N$19: now also C26.1, IC2.CATHODE, R17.1; no longer R21.1, U8.ANODE1
- net RST: now also R11.1
- net SCLK_EXT: now also R21.6; no longer U8.CATHODE2
- net SF_EXT: now also R21.5; no longer U8.CATHODE1
- net SPI1_MISO: now also R17.2; no longer IC2.CATHODE
- net SPI2_MISO: now also C27.1
- net SS_EXT: now also R21.8; no longer U8.CATHODE4
Other:
- moved on the sheet: MISO1, R11, R16, R17, R21, SCK2, U8
