File: Basisplatine/basisplatine.sch (EAGLE design)
At the start: 27 parts, among them IC1 RASPBERRY_PI_ZERO_W__V1.3_, IC2 MEGA8-AI

Commit message: added battery managment
Parts:
- added C13: 100n, rcl:C-EUC0603K
- added C14, C15, C16, C19, C20: 10u, rcl:C-EUC1206K
- added C17, C21: 120p, rcl:C-EUC0603K
- added C18: 2u2, rcl:C-EUC1206K
- added IC3: DIO5158XS8, basisplatine_lib:DIO5158XS8
- added IC4: TPS613222ADBVR, basisplatine_lib:TPS613222ADBVR
- added IC5: AP63205WU-7, basisplatine_lib:AP63205WU-7
- added J1: DCJ0202, con-jack:DCJ0202
- added JP1, JP2: (no value), pinhead:PINHD-1X2
- added L1: SRN5040TA-4R7M, basisplatine_lib:SRN5040TA-4R7M
- added Q2: NTF5P03T3G, basisplatine_lib:NTF5P03T3G
- added R10, R11, R12, R13, R14, R18, R19, R9: (no value), rcl:R-EU_R0603
- added R15: 5R, rcl:R-EU_R0603
- added R16, R17, R29, R30, R31: 10k, rcl:R-EU_R0603
- added R20, R21, R22, R23, R24, R25, R26, R28: 100R, rcl:R-EU_R0603
- added R27: 2k, rcl:R-EU_R0603
- added R8: 1218R, rcl:R-EU_R0603
- added S1: (no value), switch-omron:10-XX
- added T1: (no value), transistor:BC808-NPN-SOT23-BEC
- added U$10, U$11, U$7, U$9: SK1035-TP, basisplatine_lib:SK1035-TP
- added U$6, U$8: SRP1038C-2R2M, basisplatine_lib:SRP1038C-2R2M
Connections:
- net N$7 renamed ADC0
- net N$8 renamed ADC1
- net N$9 renamed ADC2
- new net ADC3: IC2.PC3(ADC3), R11.2, R12.1
- new net ADC4: IC2.PC4(ADC4/SDA), R13.2, R14.1
- new net ADC5: IC2.PC5(ADC5/SCL), R18.2, R19.1
- new net BOOST_EN: IC2.PD5(T1), R17.2
- new net CHARGE_EN: IC2.PD2(INT0), IC3.CE
- new net ISET: IC3.ISET, R4.1, R8.2
- new net N$1: IC4.SW, R15.2, U$6.2, U$7.A
- new net N$10: Q2.G, R16.2, T1.C
- new net N$11: R17.1, T1.B
- new net N$12: Q2.D, Q2.D_TAB, S1.S, S1.S1, U$10.A
- new net N$13: C21.2, IC5.BST
- new net N$15: IC1.GPIO_24, R22.1
- new net N$16: IC1.GPIO_23, R23.1
- new net N$17: IC1.GPIO_22, R24.1
- new net N$18: IC1.GPIO27, R25.1
- new net N$19: IC1.GPIO_18/PWM0/SPI1_CS0, R26.1
- new net N$20: IC2.PB1(OC1A), R28.1
- new net N$21: IC2.PB3(MOSI/OC2), R29.1
- new net N$22: IC2.PB4(MISO), R30.1
- new net N$23: IC2.PB5(SCK), R31.1
- new net N$5: IC5.EN, IC5.VIN, U$11.C
- new net N$7: C17.1, R15.1
- new net N$8: C16.1, C17.2, IC4.VOUT, U$7.C, U$8.1
- new net N$9: C18.1, U$10.C, U$6.1, U$9.C
- new net SHUTDOWN: IC1.GPIO6/GPCLK2, IC2.PD6(AIN0)
- new net SPI_CLK_R: IC1.GPIO_11/SPI0_SCLK, R20.2, R31.2
- new net SPI_MOSI_R: IC1.GPIO_10/SPI0_MOSI, R21.1, R29.2
- new net STATUS_CHARGE: IC2.PD3(INT1), IC3.!CHRG
- new net STATUS_DONE: IC2.PD4(XCK/T0), IC3.!DONE
- new net TEMP: IC3.TEMP, JP1.2, R10.2, R9.1
- new net VIN: C20.1, IC3.VIN, IC5.FB, L1.2, R13.1, R9.2, U$9.A
- new net VJACK: C13.2, C14.1, J1.1, R18.1, U$11.A
- net +3V3: now also R27.2
- net +5V: now also C19.1, U$8.2
- net CLOCK_EN: now also IC1.GPIO_17/SPI1_CS1
- net GND: now also C13.1, C14.2, C15.2, C16.2, C18.2, C19.2, C20.2, IC3.GND, IC3.THERM, IC4.GND, IC5.GND, J1.2, J1.3, JP1.1, JP2.2, R10.1, R12.2, R14.2, R19.2, R8.1, T1.E
- net N$6: now also C21.1, IC5.SW, L1.1; no longer IC1.GPIO_17/SPI1_CS1
- net SAMPLE: now also R28.2; no longer IC2.PB1(OC1A)
- net SPI_CLK: now also R20.1; no longer IC1.GPIO_11/SPI0_SCLK, IC2.PB5(SCK)
- net SPI_MISO: now also R27.1, R30.2; no longer IC2.PB4(MISO)
- net SPI_MOSI: now also R21.2; no longer IC1.GPIO_10/SPI0_MOSI, IC2.PB3(MOSI/OC2)
- net SS1: now also R22.2; no longer IC1.GPIO_24
- net SS2: now also R23.2; no longer IC1.GPIO_23
- net SS3: now also R24.2; no longer IC1.GPIO_22
- net SS4: now also R25.2; no longer IC1.GPIO27
- net SS5: now also R26.2; no longer IC1.GPIO_18/PWM0/SPI1_CS0
- net VBAT: now also C15.1, IC3.BAT, JP2.1, Q2.S, R11.1, R16.1, S1.P, S1.P1; no longer R4.1
Other:
- note added: "NTC"
- note added: "Startbutton"

Commit message: Added dampening Cs on SPI and RJ45
Parts:
- added C22: (no value), rcl:C-EUC1206
- added C23, C24, C25, C26: 2u2, rcl:C-EUC1206K
- added C27, C28, C29, C30, C31: 100n, rcl:C-EUC0603K
- added C32, C33, C34, C35, C36, C37, C38, C39, C40, C41, C42, C43, C44, C45, C46, C47, C48: (no value), rcl:C-EUC0603K
- added J2, J3, J4, J5, J6: 54601-908WPLF, basisplatine_lib:54601-908WPLF
- added R32, R33, R34, R35, R36, R37: 100R, rcl:R-EU_R0603
- added T2: (no value), transistor:BC808-NPN-SOT23-BEC
Connections:
- removed net N$21: IC2.PB3(MOSI/OC2), R29.1
- removed net N$23: IC2.PB5(SCK), R31.1
- new net N$14: R30.2, T2.B
- new net N$24: IC1.GPIO5//GPCLK1, R32.2
- new net N$25: IC1.GPIO12/PWM0, R37.2
- new net N$26: IC1.GPIO13/PWM1, R36.2
- new net N$27: IC1.GPIO19/SPI0_MISO1/PWM1, R35.2
- new net N$28: IC1.GPIO16/SPI1_CS2, R34.2
- new net N$29: IC1.GPIO26, R33.2
- new net SPI_CLK_ATMEGA: C48.2, IC2.PB5(SCK), R31.1
- new net SPI_MOSI_ATMEGA: C47.2, IC2.PB3(MOSI/OC2), R29.1
- new net SS10: C42.2, J6.2, R37.1
- new net SS6: C38.2, J2.2, R33.1
- new net SS7: C39.2, J3.2, R34.1
- new net SS8: C40.2, J4.2, R35.1
- new net SS9: C41.2, J5.2, R36.1
- net +3V3: now also R1.1
- net +5V: now also C22.1, C23.1, C24.1, C25.1, C26.1, C27.1, C28.1, C29.1, C30.1, C31.1, J2.1, J3.1, J4.1, J5.1, J6.1
- net CLOCK_EN: no longer IC1.GPIO_17/SPI1_CS1
- net GND: now also C22.2, C23.2, C24.2, C25.2, C26.2, C27.2, C28.2, C29.2, C30.2, C31.2, C32.1, C33.1, C34.1, C35.1, C36.1, C37.1, C38.1, C39.1, C40.1, C41.1, C42.1, C43.1, C44.1, C45.1, C46.1, C47.1, C48.1, J2.5, J2.8, J3.5, J3.8, J4.5, J4.8, J5.5, J5.8, J6.5, J6.8, T2.E; no longer R1.1
- net SAMPLE: now also C46.2, J2.6, J3.6, J4.6, J5.6, J6.6
- net SPI_CLK: now also C43.2, J2.4, J3.4, J4.4, J5.4, J6.4
- net SPI_MISO: now also C44.2, J2.7, J3.7, J4.7, J5.7, J6.7, T2.C; no longer R30.2
- net SPI_MOSI: now also C45.2, J2.3, J3.3, J4.3, J5.3, J6.3
- net SS0: now also C32.2, R32.1; no longer IC1.GPIO5//GPCLK1
- net SS1: now also C33.2
- net SS2: now also C34.2
- net SS3: now also C35.2
- net SS4: now also C36.2
- net SS5: now also C37.2
Other:
- note added: "COM-Dampener"
- moved on the sheet: R29, R31

Commit message: Added Stueckliste, Taster, LED
Parts:
- added LED1: ASMB-UTF0-0D20B, basisplatine_lib:ASMB-UTF0-0D20B
- added R38, R39, R40: 100R, rcl:R-EU_R0603
- added S2: (no value), switch-omron:10-XX
- added U$12: SK1035-TP, basisplatine_lib:SK1035-TP
- C1, C22: value (none) -> 10u
- C18, C2, C23, C24, C25, C26, C3, C4, C5: value 2u2 -> 10u
- R11, R13, R2, R3: value (none) -> 82k
- R12, R14, R19, R4, R5, R6, R7: value (none) -> 10k
- R18: value (none) -> 270k
Connections:
- net SHUTDOWN renamed RUNNING
- removed net N$10: Q2.G, R16.2, T1.C
- new net LED_BLUE: IC1.GPIO_4/GPCLK0, R40.2
- new net LED_GREEN: IC1.GPIO_3/[I2C]_SCL, R39.2
- new net LED_RED: IC1.GPIO_2/[I2C]_SDA, R38.2
- new net N$21: IC1.GPIO21/SPI0_SCLK1, S2.P, S2.P1
- new net N$23: Q2.G, R16.2, T1.C, U$12.A
- new net N$30: LED1.RED_ANODE, R38.1
- new net N$31: LED1.GREEN_ANODE, R39.1
- new net N$32: LED1.BLUE_ANODE, R40.1
- new net RESET_PI: IC1.RUN_1, IC2.PD7(AIN1)
- new net START_STOPBUTTON: IC2.PB0(ICP), S1.P, S1.P1, U$12.C
- net GND: now also LED1.BLUE_CATHODE, LED1.GREEN_CATHODE, LED1.RED_CATHODE, S1.S, S1.S1, S2.S, S2.S1
- net N$12: no longer S1.S, S1.S1
- net VBAT: no longer S1.P, S1.P1
Other:
- moved on the sheet: S1

Commit message: Added 3,3V and vias to Basisplatine, ...
Parts:
- removed U$7: SK1035-TP, basisplatine_lib:SK1035-TP
- added C49, C50, C51, C52, C53, C54, C55, C56, C57, C58: 100n, rcl:C-EUC0603K
- added D1: SBRT10U50SP5-13, basisplatine_lib:SBRT10U50SP5-13
Connections:
- net +3V3: now also C49.1, C50.1, C51.1, C52.1, C53.1, C54.1, C55.1, C56.1, C57.1, C58.1, J2.8, J3.8, J4.8, J5.8, J6.8, U$1.3.3V1, U$1.3.3V2, U$2.3.3V1, U$2.3.3V2, U$3.3.3V1, U$3.3.3V2, U$4.3.3V1, U$4.3.3V2, U$5.3.3V1, U$5.3.3V2
- net GND: now also C49.2, C50.2, C51.2, C52.2, C53.2, C54.2, C55.2, C56.2, C57.2, C58.2; no longer J2.8, J3.8, J4.8, J5.8, J6.8
- net N$1: now also D1.A_1, D1.A_2; no longer U$7.A
- net N$8: now also D1.K; no longer U$7.C
