File: Steckkarte/Steckkarte2/Steckkarte.brd (EAGLE design)
At the start: 63 x 92.5 mm, 99 parts, among them IC1 OPA2333D, IC2 TLP2768A_TP,E, U1 STM32L412CBT6, U2 LP5907QMFX-3.3Q1, U3 REF5030AIDR, U4 RFM-0505S, U5 Value, U6 TLV4110IDGNR, U7 W25Q64JVSSIQ, U8 ACSL-6400-00TE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

Commit message: steckkarte die 2.te
Parts:
- added R12, R26, R27: 160, rcl:R0603
- C1: value 2.2µ -> 4,7µ
- C15: value 100µF -> 100n; device resistor:C1206K -> rcl:C0603K
- C2: value 1.8µ -> 2.2µ; device rcl:C1206K -> rcl:C0603K
- R17: value 150 -> 160
- R21: value EXB-V8V103JV_200 -> 160; device EXB-V8V103:EXBV8V -> rcl:R0603
- moved I/O5 57.0 mm to (58.0, 55.5)
- moved R20 56.9 mm to (58.0, 60.0)
- moved I/O3 56.8 mm to (58.0, 72.5)
- moved I/O4 56.8 mm to (58.0, 64.5)
- moved R19 56.8 mm to (58.0, 68.5)
- moved V-I 49.0 mm to (52.5, 53.0)
- moved D1 46.1 mm to (52.1, 69.4), turned to 270 degrees
- moved R7 38.9 mm to (45.0, 70.0), turned to 270 degrees
- moved U6 37.9 mm to (48.5, 56.4), turned to 180 degrees
- moved V- 37.7 mm to (52.0, 61.5), turned to 180 degrees
- moved C23 34.8 mm to (38.5, 61.2), turned to 270 degrees
- moved ADJ 33.1 mm to (40.5, 67.0)
- moved CR1 33.1 mm to (43.9, 64.0)
- moved R24 32.7 mm to (48.5, 70.0)
- moved R8 31.0 mm to (41.9, 70.0)
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Connections:
- net +3V3: now also C19.2, U9.5; no longer C23.1, CR1.4
- net +5V: now also C23.1, CR1.4; no longer C19.2, U9.5
- net DAC1_EN: now also U1.42; no longer U1.22
- net MOSI_EXT: now also R26.2; no longer R21.7
- net N$16: now also R26.1; no longer R21.2
- net N$17: now also R21.1; no longer R21.3
- net N$18: now also R12.1; no longer R21.4
- net N$9: now also R27.1; no longer R21.1
- net SCLK_EXT: now also R21.2; no longer R21.6
- net SF_EXT: now also R12.2; no longer R21.5
- net SS_EXT: now also R27.2; no longer R21.8
Routing:
- net DAC1_EN: track 65.6 -> 22.7 mm, vias 2 -> 0
- net +5V: track 202.6 -> 164.5 mm, vias 6 -> 5
- net GND5: track 266.5 -> 231.2 mm, vias 142 -> 141
- net DAC1: track 67.0 -> 37.0 mm
- net +3V3: track 213.7 -> 199.6 mm, vias 10 -> 7
- net 5V_EXT: track 79.2 -> 65.6 mm, vias 2 -> 3
- net LED: track 41.4 -> 31.9 mm, vias 0 -> 2
- net SS_EXT: track 7.92 -> 17.0 mm
- net LSP3: track 39.6 -> 32.3 mm
- net 3.3V_EXT: track 41.5 -> 35.5 mm
- net LSP5: track 17.8 -> 23.2 mm
- net N$9: track 9.53 -> 4.67 mm
- net N$16: track 8.81 -> 4.07 mm
- net MOSI_EXT: track 4.71 -> 9.42 mm
- net SCLK_EXT: track 4.79 -> 9.43 mm
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Other:
- board size 63 x 92.5 mm -> 63 x 76.5 mm
- board text added: "Steckkarte MB2000 v.1.0"
- board text removed: "Steckkarte Messbox 2000 v1.0"
- board text removed: "and partly Johannes Wittmann"
- board text removed: "blame Timo Erdmannsdörfer"
