File: Steckkarte/Steckkarte2/Steckkarte.sch (EAGLE design)
At the start: 99 parts, among them IC1 OPA2333D, IC2 TLP2768A_TP,E, U1 STM32L412CBT6, U2 LP5907QMFX-3.3Q1, U3 REF5030AIDR, U4 RFM-0505S, U5 Value, U6 TLV4110IDGNR, U7 W25Q64JVSSIQ, U8 ACSL-6400-00TE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

Commit message: steckkarte die 2.te
Parts:
- added R12, R26, R27: 160, rcl:R-EU_R0603
- C1: value 2.2µ -> 4,7µ
- C15: value 100µF -> 100n; device resistor:C-EUC1206K -> rcl:C-EUC0603K
- C2: value 1.8µ -> 2.2µ; device rcl:C-EUC1206K -> rcl:C-EUC0603K
- R17: value 150 -> 160
- R21: value EXB-V8V103JV_200 -> 160; device EXB-V8V103:EXB-V8V103JV -> rcl:R-EU_R0603
Connections:
- net +3V3: now also C19.2, U9.V+; no longer C23.1, CR1.V+
- net +5V: now also C23.1, CR1.V+; no longer C19.2, U9.V+
- net DAC1_EN: now also U1.PB6; no longer U1.PB11
- net MOSI_EXT: now also R26.2; no longer R21.7
- net N$16: now also R26.1; no longer R21.2
- net N$17: now also R21.1; no longer R21.3
- net N$18: now also R12.1; no longer R21.4
- net N$9: now also R27.1; no longer R21.1
- net SCLK_EXT: now also R21.2; no longer R21.6
- net SF_EXT: now also R12.2; no longer R21.5
- net SS_EXT: now also R27.2; no longer R21.8
Other:
- moved on the sheet: I/O1, I/O2, R19
